File: hardware-ESPC3Supermini-handsoldered/ESP32C3_Supermini_LG_climate_contoller-handsoldered.kicad_pcb (KiCad board)
At the start: 2 copper layers, 25 x 21.6 mm, 18 parts, among them J1 Conn_01x01_Pin, J2 Conn_01x01_Pin, J3 Conn_01x01_Pin, U1 ESP32-C3_SUPERMINI, U2 TPS560200, U4 TJA1027T

Commit message: moved designators
Parts:
- renumbered C3 to C1, C4 to C3, C5 to C4, C1 to C5, U2 to U1, U4 to U2, U1 to U3
